Commit message: fix tf tree

File: rc_car_navigation/urdf/rc_car.urdf (robot description, URDF)
Before this commit: robot rc_car, 2 links, 1 joints
Joints:
- removed joint base_joint
- added joint base_footprint_joint: type fixed, parent base_link, child base_footprint, origin xyz=0 0 -0.05 rpy=0 0 0
